File: pcb/MIDIPak_v2.brd (EAGLE design)
At the start: 61 x 88.3 mm, 41 parts, among them IC1 74LS133N, IC3 74LS138N, IC4 68B50, IC5 74LS04N, IC6 74LS161, Q1 4MHz, T1 2N2222/3904, X1 MIDI_IN, X2 MIDI_THRU, X3 MIDI_OUT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

Commit message: Fixed polarity issues with LED signals
Parts:
- moved T1 1.27 mm to (8.89, 63.5), turned to 270 degrees
- turned LED1 to 180 degrees
- turned LED2 to 180 degrees
- turned LED3 to 180 degrees
- turned R11 to 270 degrees
- turned R12 to 270 degrees
- turned R13 to 270 degrees
Connections:
- removed net N$25: LED1.A, R11.2
- removed net N$26: LED2.A, R12.2
- removed net N$29: LED3.A, R13.2
- new net N$18: LED2.K, R12.1
- new net N$21: LED1.K, R11.1
- new net N$22: LED3.K, R13.1
- net GND: now also R11.2, R12.2, R13.2; no longer T1.3
- net LED_OUT: now also LED2.A; no longer LED2.K
- net LED_THRU: now also LED3.A; no longer LED3.K
- net N$2: now also LED1.A, T1.3; no longer LED1.K, T1.1
- net VCC: now also T1.1; no longer R11.1, R12.1, R13.1
Routing:
- net N$29: track 7.14 -> 0.00 mm
- net N$25: track 7.14 -> 0.00 mm
- net N$22: track 0.00 -> 7.14 mm
- net N$21: track 0.00 -> 7.14 mm
- net N$26: track 7.14 -> 0.00 mm
- net N$18: track 0.00 -> 7.14 mm
- net VCC: track 260.2 -> 255.8 mm
- net RXD: track 85.7 -> 81.6 mm, vias 0 -> 1
- net N$20: track 9.35 -> 6.50 mm
- net N$2: track 13.8 -> 13.2 mm
Changed lines of the file:
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@@
 </element>
 <element name="C7" library="rcl" package="C025-025X050" value="" x="24.13" y="61.595" rot="R180"/>
-<element name="LED1" library="led" package="LED3MM" value="" x="20.32" y="66.04"/>
-<element name="LED2" library="led" package="LED3MM" value="" x="0" y="66.04"/>
-<element name="LED3" library="led" package="LED3MM" value="" x="-20.32" y="66.04"/>
-<element name="R11" library="resistor" package="0204/7" value="220R" x="12.7" y="64.135" rot="R90"/>
-<element name="R12" library="resistor" package="0204/7" value="220R" x="-7.62" y="64.135" rot="R90"/>
-<element name="R13" library="resistor" package="0204/7" value="220R" x="-27.94" y="64.135" rot="R90"/>
+<element name="LED1" library="led" package="LED3MM" value="" x="20.32" y="66.04" rot="R180"/>
+<element name="LED2" library="led" package="LED3MM" value="" x="0" y="66.04" rot="R180"/>
+<element name="LED3" library="led" package="LED3MM" value="" x="-20.32" y="66.04" rot="R180"/>
+<element name="R11" library="resistor" package="0204/7" value="220R" x="12.7" y="64.135" rot="R270"/>
+<element name="R12" library="resistor" package="0204/7" value="220R" x="-7.62" y="64.135" rot="R270"/>
+<element name="R13" library="resistor" package="0204/7" value="220R" x="-27.94" y="64.135" rot="R270"/>
 <element name="R14" library="resistor" package="0204/7" value="10K" x="12.7" y="53.975" rot="R90"/>
-<element name="T1" library="transistor" package="TO92" value="2N2222/3904" x="8.89" y="64.77" rot="R90"/>
+<element name="T1" library="transistor" package="TO92" value="2N2222/3904" x="8.89" y="63.5" rot="R270"/>
 <element name="JP1" library="jumper-jlb" package="JP2" value="" x="0" y="53.975" rot="R90"/>
 <element name="JP2" library="jumper-jlb" package="JP1" value="" x="-11.43" y="67.945" rot="R90"/>
@@
 <contactref element="OK1" pad="5"/>
 <contactref element="C7" pad="2"/>
-<contactref element="T1" pad="3"/>
 <contactref element="JP2" pad="2"/>
+<contactref element="R13" pad="2"/>
+<contactref element="R12" pad="2"/>
+<contactref element="R11" pad="2"/>
 </signal>
 <signal name="VCC">
@@
 <wire x1="-24.13" y1="59.055" x2="-25.4" y2="60.325" width="0.6096" layer="1"/>
 <wire x1="-25.4" y1="60.325" x2="-25.4" y2="62.23" width="0.6096" layer="16"/>
-<wire x1="-25.4" y1="62.23" x2="-7.62" y2="62.23" width="0.6096" layer="16"/>
-<wire x1="-7.62" y1="62.23" x2="-5.08" y2="62.23" width="0.6096" layer="16"/>
+<wire x1="-25.4" y1="62.23" x2="-5.08" y2="62.23" width="0.6096" layer="16"/>
 <wire x1="-5.08" y1="62.23" x2="-5.08" y2="60.325" width="0.254" layer="16"/>
 <wire x1="15.24" y1="41.275" x2="12.7" y2="41.275" width="0.6096" layer="1"/>
@@
 <wire x1="16.51" y1="46.99" x2="12.7" y2="46.99" width="0.6096" layer="1"/>
 <wire x1="12.7" y1="46.99" x2="12.7" y2="45.72" width="0.6096" layer="1"/>
-<wire x1="12.7" y1="62.23" x2="12.7" y2="60.325" width="0.6096" layer="16"/>
-<wire x1="-5.08" y1="62.23" x2="12.7" y2="62.23" width="0.6096" layer="16"/>
+<wire x1="-5.08" y1="62.23" x2="8.89" y2="62.23" width="0.6096" layer="16"/>
+<wire x1="8.89" y1="62.23" x2="12.7" y2="62.23" width="0.6096" layer="16"/>
 <wire x1="-6.35" y1="22.225" x2="-6.35" y2="24.4475" width="0.6096" layer="16"/>
 <wire x1="-6.35" y1="24.4475" x2="-1.27" y2="24.4475" width="0.6096" layer="16"/>
@@
 <wire x1="25.4" y1="57.785" x2="25.4" y2="46.99" width="0.6096" layer="1"/>
 <wire x1="27.94" y1="57.785" x2="25.4" y2="57.785" width="0.6096" layer="1"/>
-<contactref element="R12" pad="1"/>
-<contactref element="R13" pad="1"/>
-<contactref element="R11" pad="1"/>
-<wire x1="-27.94" y1="60.325" x2="-25.4" y2="60.325" width="0.254" layer="1"/>
-<wire x1="-7.62" y1="60.325" x2="-7.62" y2="62.23" width="0.254" layer="16"/>
-<wire x1="12.7" y1="60.325" x2="15.24" y2="57.785" width="0.6096" layer="16"/>
 <wire x1="15.24" y1="57.785" x2="16.51" y2="56.515" width="0.6096" layer="1"/>
 <wire x1="16.51" y1="56.515" x2="16.51" y2="46.99" width="0.6096" layer="1"/>
+<contactref element="T1" pad="1"/>
+<wire x1="12.7" y1="62.23" x2="13.97" y2="60.96" width="0.6096" layer="16"/>
+<wire x1="13.97" y1="60.96" x2="13.97" y2="59.055" width="0.6096" layer="16"/>
+<wire x1="13.97" y1="59.055" x2="15.24" y2="57.785" width="0.6096" layer="16"/>
 </signal>
 <signal name="N$1">
@@
 <wire x1="-21.59" y1="22.225" x2="-21.59" y2="35.8775" width="0.254" layer="1"/>
 <wire x1="-21.59" y1="35.8775" x2="-20.32" y2="37.1475" width="0.254" layer="1"/>
-<wire x1="-20.32" y1="37.1475" x2="-20.32" y2="42.545" width="0.254" layer="1"/>
-<wire x1="-20.32" y1="42.545" x2="-22.86" y2="45.085" width="0.254" layer="1"/>
-<wire x1="-22.86" y1="45.085" x2="-22.86" y2="48.895" width="0.254" layer="1"/>
+<wire x1="-20.32" y1="37.1475" x2="-20.32" y2="47.9425" width="0.254" layer="1"/>
+<wire x1="-20.32" y1="47.9425" x2="-19.3675" y2="48.895" width="0.254" layer="1"/>
 <wire x1="24.13" y1="48.895" x2="15.24" y2="48.895" width="0.254" layer="16"/>
 <wire x1="15.24" y1="48.895" x2="12.7" y2="48.895" width="0.254" layer="16"/>
 <wire x1="12.7" y1="48.895" x2="0" y2="48.895" width="0.254" layer="16"/>
-<wire x1="0" y1="48.895" x2="-22.86" y2="48.895" width="0.254" layer="16"/>
+<wire x1="0" y1="48.895" x2="-19.3675" y2="48.895" width="0.254" layer="16"/>
 <wire x1="15.24" y1="50.165" x2="15.24" y2="48.895" width="0.254" layer="16"/>
 <contactref element="OK1" pad="6"/>
@@
 <contactref element="JP1" pad="1"/>
 <wire x1="0" y1="51.435" x2="0" y2="48.895" width="0.254" layer="16"/>
-<wire x1="-22.86" y1="48.895" x2="-22.86" y2="48.895" width="0" layer="19" extent="1-16"/>
+<via x="-19.3675" y="48.895" extent="1-16" drill="0.3048"/>
 </signal>
 <signal name="N$15">
@@
 <contactref element="R14" pad="2"/>
 <contactref element="T1" pad="2"/>
-<wire x1="6.985" y1="64.77" x2="6.985" y2="63.5" width="0.254" layer="1"/>
-<wire x1="6.985" y1="63.5" x2="12.7" y2="57.785" width="0.254" layer="1"/>
-</signal>
-<signal name="N$25">
-<contactref element="R11" pad="2"/>
-<contactref element="LED1" pad="A"/>
-<wire x1="12.7" y1="67.945" x2="14.605" y2="66.04" width="0.254" layer="1"/>
-<wire x1="14.605" y1="66.04" x2="19.05" y2="66.04" width="0.254" layer="1"/>
-</signal>
-<signal name="N$26">
-<contactref element="R12" pad="2"/>
-<contactref element="LED2" pad="A"/>
-<wire x1="-7.62" y1="67.945" x2="-5.715" y2="66.04" width="0.254" layer="1"/>
-<wire x1="-5.715" y1="66.04" x2="-1.27" y2="66.04" width="0.254" layer="1"/>
-</signal>
-<signal name="N$29">
-<contactref element="R13" pad="2"/>
-<contactref element="LED3" pad="A"/>
-<wire x1="-27.94" y1="67.945" x2="-26.035" y2="66.04" width="0.254" layer="1"/>
-<wire x1="-26.035" y1="66.04" x2="-21.59" y2="66.04" width="0.254" layer="1"/>
+<wire x1="10.795" y1="63.5" x2="10.795" y2="59.69" width="0.254" layer="1"/>
+<wire x1="10.795" y1="59.69" x2="12.7" y2="57.785" width="0.254" layer="1"/>
 </signal>
 <signal name="LED_OUT">
-<contactref element="LED2" pad="K"/>
 <contactref element="IC5" pad="4"/>
 <contactref element="IC5" pad="11"/>
@@
 <wire x1="-15.875" y1="57.785" x2="-10.16" y2="63.5" width="0.254" layer="1"/>
 <wire x1="-10.16" y1="63.5" x2="-1.27" y2="63.5" width="0.254" layer="1"/>
-<wire x1="-1.27" y1="63.5" x2="1.27" y2="66.04" width="0.254" layer="1"/>
+<contactref element="LED2" pad="A"/>
+<wire x1="1.27" y1="66.04" x2="-1.27" y2="63.5" width="0.254" layer="1"/>
 </signal>
 <signal name="LED_THRU">
-<contactref element="LED3" pad="K"/>
 <contactref element="IC5" pad="2"/>
 <contactref element="IC5" pad="13"/>
 <wire x1="-21.59" y1="57.785" x2="-21.59" y2="50.165" width="0.254" layer="1"/>
 <wire x1="-21.59" y1="57.785" x2="-19.05" y2="60.325" width="0.254" layer="1"/>
+<contactref element="LED3" pad="A"/>
 <wire x1="-19.05" y1="60.325" x2="-19.05" y2="66.04" width="0.254" layer="1"/>
-</signal>
-<signal name="N$2">
-<contactref element="LED1" pad="K"/>
-<contactref element="T1" pad="1"/>
-<wire x1="8.89" y1="66.04" x2="10.16" y2="64.77" width="0.254" layer="1"/>
-<wire x1="10.16" y1="64.77" x2="20.32" y2="64.77" width="0.254" layer="1"/>
-<wire x1="20.32" y1="64.77" x2="21.59" y2="66.04" width="0.254" layer="1"/>
 </signal>
 <signal name="N$12">
@@
 <wire x1="-10.16" y1="67.945" x2="-10.16" y2="85.725" width="0.254" layer="1"/>
 </signal>
+<signal name="N$22">
+<contactref element="R13" pad="1"/>
+<contactref element="LED3" pad="K"/>
+<wire x1="-27.94" y1="67.945" x2="-26.035" y2="66.04" width="0.254" layer="1"/>
+<wire x1="-26.035" y1="66.04" x2="-21.59" y2="66.04" width="0.254" layer="1"/>
+</signal>
+<signal name="N$18">
+<contactref element="LED2" pad="K"/>
+<contactref element="R12" pad="1"/>
+<wire x1="-7.62" y1="67.945" x2="-5.715" y2="66.04" width="0.254" layer="1"/>
+<wire x1="-5.715" y1="66.04" x2="-1.27" y2="66.04" width="0.254" layer="1"/>
+</signal>
+<signal name="N$2">
+<contactref element="T1" pad="3"/>
+<contactref element="LED1" pad="A"/>
+<wire x1="21.59" y1="66.04" x2="20.32" y2="64.77" width="0.254" layer="1"/>
+<wire x1="20.32" y1="64.77" x2="8.89" y2="64.77" width="0.254" layer="1"/>
+</signal>
+<signal name="N$21">
+<contactref element="LED1" pad="K"/>
+<contactref element="R11" pad="1"/>
+<wire x1="12.7" y1="67.945" x2="14.605" y2="66.04" width="0.254" layer="1"/>
+<wire x1="14.605" y1="66.04" x2="19.05" y2="66.04" width="0.254" layer="1"/>
+</signal>
 </signals>
