File: pcb/MIDIPak_v3.brd (EAGLE design)
At the start: 61 x 88.3 mm, 38 parts, among them IC1 74LS133N, IC3 74LS138N, IC4 68B50, IC5 74LS04N, IC6 74*161, X1 MIDI_IN, X2 MIDI_THRU, X3 MIDI_OUT, X4 EXPANSION_PORT_COCO

Commit message: Fixed polarity issues with LED signals
Parts:
- turned IN to 90 degrees
- turned LED1 to 180 degrees
- turned LED2 to 180 degrees
- turned LED3 to 180 degrees
- turned OUT to 90 degrees
- turned THRU to 90 degrees
Connections:
- removed net N$19: LED3.A, R10.1, THRU.1
- new net N$17: LED2.K, OUT.2, R6.1
- net GND: now also R10.2, R3.2, R6.2
- net LED_IN: now also IN.1, LED1.A; no longer IN.2, LED1.K
- net LED_OUT: now also LED2.A, OUT.1; no longer LED2.K, OUT.2
- net LED_THRU: now also LED3.A, THRU.1; no longer LED3.K, THRU.2
- net N$12: now also IN.2, LED1.K; no longer IN.1, LED1.A
- net N$18: now also LED3.K, R10.1, THRU.2; no longer LED2.A, OUT.1, R6.1
- net VCC: no longer R10.2, R3.2, R6.2
Routing:
- net N$19: track 10.9 -> 0.00 mm
- net N$17: track 0.00 -> 10.9 mm
- net VCC: track 263.7 -> 258.6 mm
Changed lines of the file:
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@@
 <attribute name="OC_NEWARK" value="unknown" x="8.89" y="53.975" size="1.778" layer="27" display="off"/>
 </element>
-<element name="LED1" library="led" package="LED3MM" value="" x="20.32" y="66.04"/>
-<element name="LED2" library="led" package="LED3MM" value="" x="0" y="66.04"/>
-<element name="LED3" library="led" package="LED3MM" value="" x="-20.32" y="66.04"/>
+<element name="LED1" library="led" package="LED3MM" value="" x="20.32" y="66.04" rot="R180"/>
+<element name="LED2" library="led" package="LED3MM" value="" x="0" y="66.04" rot="R180"/>
+<element name="LED3" library="led" package="LED3MM" value="" x="-20.32" y="66.04" rot="R180"/>
 <element name="JP1" library="jumper-jlb" package="JP2" value="" x="0" y="53.975" rot="R90"/>
 <element name="R3" library="resistor" package="0204/7" value="220" x="12.7" y="64.135" rot="R270"/>
@@
 <element name="JP2" library="jumper-jlb" package="JP1" value="" x="-11.43" y="67.6275" rot="R90"/>
 <element name="C6" library="rcl" package="C025-025X050" value="" x="25.4" y="62.865" rot="R90"/>
-<element name="IN" library="jumper-jlb" package="JP1" value="" x="20.32" y="62.23" rot="R270"/>
-<element name="OUT" library="jumper-jlb" package="JP1" value="" x="0" y="62.23" rot="R270"/>
-<element name="THRU" library="jumper-jlb" package="JP1" value="" x="-20.32" y="62.23" rot="R270"/>
+<element name="IN" library="jumper-jlb" package="JP1" value="" x="20.32" y="62.23" rot="R90"/>
+<element name="OUT" library="jumper-jlb" package="JP1" value="" x="0" y="62.23" rot="R90"/>
+<element name="THRU" library="jumper-jlb" package="JP1" value="" x="-20.32" y="62.23" rot="R90"/>
 </elements>
 <signals>
@@
 <contactref element="IC6" pad="5"/>
 <contactref element="IC6" pad="4"/>
+<contactref element="R3" pad="2"/>
+<contactref element="R6" pad="2"/>
+<contactref element="R10" pad="2"/>
 </signal>
 <signal name="VCC">
@@
 <wire x1="-5.08" y1="59.055" x2="-5.08" y2="60.325" width="0.254" layer="1"/>
 <wire x1="5.08" y1="57.785" x2="6.35" y2="57.785" width="0.6096" layer="1"/>
-<contactref element="R3" pad="2"/>
-<contactref element="R6" pad="2"/>
-<contactref element="R10" pad="2"/>
-<wire x1="12.7" y1="60.325" x2="12.7" y2="59.055" width="0.254" layer="1"/>
-<wire x1="-7.62" y1="60.325" x2="-7.62" y2="59.055" width="0.254" layer="1"/>
-<wire x1="-27.94" y1="60.325" x2="-25.4" y2="60.325" width="0.254" layer="1"/>
 <contactref element="OK1" pad="8"/>
 <contactref element="C6" pad="1"/>
@@
 <wire x1="-19.05" y1="55.245" x2="-24.13" y2="50.165" width="0.254" layer="16"/>
 </signal>
-<signal name="N$18">
-<contactref element="R6" pad="1"/>
-<contactref element="LED2" pad="A"/>
-<wire x1="-7.62" y1="67.945" x2="-5.715" y2="66.04" width="0.254" layer="1"/>
-<wire x1="-5.715" y1="66.04" x2="-1.27" y2="66.04" width="0.254" layer="1"/>
-<contactref element="OUT" pad="1"/>
-<wire x1="-1.27" y1="62.23" x2="-1.27" y2="66.04" width="0.254" layer="1"/>
-</signal>
-<signal name="N$19">
-<contactref element="R10" pad="1"/>
-<contactref element="LED3" pad="A"/>
-<wire x1="-27.94" y1="67.945" x2="-26.035" y2="66.04" width="0.254" layer="1"/>
-<wire x1="-26.035" y1="66.04" x2="-21.59" y2="66.04" width="0.254" layer="1"/>
-<contactref element="THRU" pad="1"/>
-<wire x1="-21.59" y1="62.23" x2="-21.59" y2="66.04" width="0.254" layer="16"/>
-</signal>
 <signal name="LED_IN">
-<contactref element="LED1" pad="K"/>
 <contactref element="IC5" pad="8"/>
 <wire x1="-8.89" y1="57.785" x2="-7.62" y2="59.055" width="0.254" layer="16"/>
@@
 <wire x1="1.905" y1="60.96" x2="4.445" y2="63.5" width="0.254" layer="16"/>
 <wire x1="4.445" y1="63.5" x2="19.05" y2="63.5" width="0.254" layer="16"/>
+<contactref element="IN" pad="1"/>
+<contactref element="LED1" pad="A"/>
+<wire x1="21.59" y1="62.23" x2="21.59" y2="66.04" width="0.254" layer="1"/>
 <wire x1="19.05" y1="63.5" x2="21.59" y2="66.04" width="0.254" layer="16"/>
-<contactref element="IN" pad="2"/>
-<wire x1="21.59" y1="62.23" x2="21.59" y2="66.04" width="0.254" layer="1"/>
 </signal>
 <signal name="LED_OUT">
-<contactref element="LED2" pad="K"/>
 <contactref element="IC5" pad="4"/>
 <contactref element="IC5" pad="11"/>
 <wire x1="-16.51" y1="57.785" x2="-16.51" y2="50.165" width="0.254" layer="1"/>
-<wire x1="1.27" y1="66.04" x2="-1.27" y2="63.5" width="0.254" layer="16"/>
 <wire x1="-1.27" y1="63.5" x2="-10.16" y2="63.5" width="0.254" layer="16"/>
 <wire x1="-10.16" y1="63.5" x2="-15.875" y2="57.785" width="0.254" layer="16"/>
 <wire x1="-15.875" y1="57.785" x2="-16.51" y2="57.785" width="0.254" layer="16"/>
-<contactref element="OUT" pad="2"/>
+<contactref element="LED2" pad="A"/>
+<contactref element="OUT" pad="1"/>
 <wire x1="1.27" y1="62.23" x2="1.27" y2="66.04" width="0.254" layer="1"/>
+<wire x1="-1.27" y1="63.5" x2="1.27" y2="66.04" width="0.254" layer="16"/>
 </signal>
 <signal name="LED_THRU">
-<contactref element="LED3" pad="K"/>
 <contactref element="IC5" pad="2"/>
 <contactref element="IC5" pad="13"/>
 <wire x1="-21.59" y1="57.785" x2="-21.59" y2="50.165" width="0.254" layer="1"/>
-<wire x1="-19.05" y1="66.04" x2="-19.05" y2="62.23" width="0.254" layer="16"/>
-<wire x1="-19.05" y1="60.96" x2="-19.05" y2="60.325" width="0.254" layer="16"/>
 <wire x1="-19.05" y1="60.325" x2="-21.59" y2="57.785" width="0.254" layer="16"/>
-<contactref element="THRU" pad="2"/>
-<wire x1="-19.05" y1="62.23" x2="-19.05" y2="60.96" width="0.254" layer="16"/>
+<contactref element="LED3" pad="A"/>
+<contactref element="THRU" pad="1"/>
+<wire x1="-19.05" y1="60.325" x2="-19.05" y2="62.23" width="0.254" layer="16"/>
+<wire x1="-19.05" y1="66.04" x2="-19.05" y2="62.23" width="0.254" layer="1"/>
 </signal>
 <signal name="N$2">
@@
 </signal>
 <signal name="N$12">
-<contactref element="IN" pad="1"/>
+<contactref element="LED1" pad="K"/>
 <contactref element="R3" pad="1"/>
-<contactref element="LED1" pad="A"/>
+<contactref element="IN" pad="2"/>
 <wire x1="12.7" y1="67.945" x2="14.605" y2="66.04" width="0.254" layer="1"/>
 <wire x1="14.605" y1="66.04" x2="19.05" y2="66.04" width="0.254" layer="1"/>
-<wire x1="19.05" y1="62.23" x2="19.05" y2="66.04" width="0.254" layer="1"/>
+<wire x1="19.05" y1="66.04" x2="19.05" y2="62.23" width="0.254" layer="1"/>
+</signal>
+<signal name="N$17">
+<contactref element="LED2" pad="K"/>
+<contactref element="R6" pad="1"/>
+<contactref element="OUT" pad="2"/>
+<wire x1="-7.62" y1="67.945" x2="-5.715" y2="66.04" width="0.254" layer="1"/>
+<wire x1="-5.715" y1="66.04" x2="-1.27" y2="66.04" width="0.254" layer="1"/>
+<wire x1="-1.27" y1="66.04" x2="-1.27" y2="62.23" width="0.254" layer="1"/>
+</signal>
+<signal name="N$18">
+<contactref element="LED3" pad="K"/>
+<contactref element="R10" pad="1"/>
+<contactref element="THRU" pad="2"/>
+<wire x1="-27.94" y1="67.945" x2="-26.035" y2="66.04" width="0.254" layer="1"/>
+<wire x1="-26.035" y1="66.04" x2="-21.59" y2="66.04" width="0.254" layer="1"/>
+<wire x1="-21.59" y1="66.04" x2="-21.59" y2="62.23" width="0.254" layer="1"/>
 </signal>
 </signals>
